File: elec_2S_BMS_plus_charger/elec_BMS_plus_charger.kicad_pcb (KiCad board)
At the start: 2 copper layers, 46 x 24 mm, 52 parts, among them J1 JST -EH 2, J13 Dynamixel-3, J14 Dynamixel-3, J2 JST SH, J3 JST -EH 2, J4 JST -EH 2, J5 pico2, J6 pico2, J7 JST SH, Q1 BSZ034N04LS, Q2 BSZ034N04LS, U1 HY2120, U2 BQ25887RGE

Commit message: [update] Release A1, small batch of 15 @JLCPCB
Other:
- board text added: "ASE01203-A1"
- board text removed: "ASE01xyz-A1"
Changed lines of the file:
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@@
 	(title_block
 		(title "Grabette -  BMS + charger")
-		(date "2026-03-18")
+		(date "2026-05-05")
 		(rev "A1")
 		(company "Pollen Robotics / Hugging Face")
@@
 			)
 		)
+		(property "FT Rotation Offset" "180"
+			(at 0 0 0)
+			(unlocked yes)
+			(layer "F.Fab")
+			(hide yes)
+			(effects
+				(font
+					(size 1 1)
+					(thickness 0.15)
+				)
+			)
+		)
 		(property ki_fp_filters "Connector*:*_1x??_*")
 		(sheetname "/Power/")
@@
 			)
 		)
+		(property "FT Rotation Offset" "180"
+			(at 0 0 0)
+			(unlocked yes)
+			(layer "F.Fab")
+			(hide yes)
+			(effects
+				(font
+					(size 1 1)
+					(thickness 0.15)
+				)
+			)
+		)
 		(property ki_fp_filters "Connector*:*_1x??_*")
 		(sheetname "/Power/")
@@
 		)
 	)
-	(gr_text "ASE01xyz-A1"
+	(gr_text "ASE01203-A1"
 		(at 146.697501 60.040001 0)
 		(layer "F.SilkS" knockout)
