File: elec_2S_BMS_plus_charger/elec_BMS_plus_charger.kicad_sch (KiCad schematic)
At the start: 8 parts

Commit message: [update] Release A1, small batch of 15 @JLCPCB
Parts:
- H1: value PCB011xy -> PCB01202
Other:
- note added: "05/05/2026"
- note added: "ASE01203"
- note removed: "ASE011xy"
- note removed: "dd/mm/2026"
Changed lines of the file:
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@@
 		)
 	)
-	(text "ASE011xy"
+	(text "ASE01203"
 		(exclude_from_sim no)
 		(at 46.99 137.795 0)
@@
 		)
 	)
-	(text "dd/mm/2026"
+	(text "05/05/2026"
 		(exclude_from_sim no)
 		(at 39.37 44.45 0)
@@
 			)
 		)
-		(property "Value" "PCB011xy"
+		(property "Value" "PCB01202"
 			(at 46.99 133.985 0)
 			(effects
