File: elec_2S_BMS_plus_charger/elec_BMS_plus_charger.kicad_sch (KiCad schematic)
At the start: 8 parts

Commit message: [update] Now running test on rasp zero 2W + HAT
Other:
- note added: "ToDo: - wrong connector for 18650, should be 2 mm pitch? - also, there are inverted +/- - I2C pins are inverted! SCL/SDA - NTC10k is mandatory - Green LED is too strong"
Changed lines of the file:
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@@
+		)
+	)
+	(text "ToDo:\n - wrong connector for 18650, should be 2 mm pitch?\n - also, there are inverted +/-\n - I2C pins are inverted! SCL/SDA\n - NTC10k is mandatory\n - Green LED is too strong"
+		(exclude_from_sim no)
+		(at 27.94 91.948 0)
+		(effects
+			(font
+				(size 3 3)
+				(italic yes)
+			)
+			(justify left bottom)
 		)
 	)
