File: elec_2S_BMS_plus_charger/power.kicad_sch (KiCad schematic)
At the start: 45 parts, among them J1 JST -EH 2, J13 Dynamixel-3, J14 Dynamixel-3, J2 JST SH, J3 JST -EH 2, J4 JST -EH 2, J5 pico2, J6 pico2, J7 JST SH, Q1 BSZ034N04LS, Q2 BSZ034N04LS, U1 HY2120, U2 BQ25887RGE

Commit message: [update] Release A1, small batch of 15 @JLCPCB
Parts:
- J5, J6: FT Rotation Offset (none) -> 180
Changed lines of the file:
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@@
 	(title_block
 		(title "Grabette - BMS + charger")
-		(date "2026-03-18")
+		(date "2026-05-05")
 		(rev "A1")
 		(company "Pollen Robotics/HF")
@@
 			)
 		)
+		(property "FT Rotation Offset" "180"
+			(at 40.64 198.12 0)
+			(effects
+				(font
+					(size 1.27 1.27)
+				)
+				(hide yes)
+			)
+		)
 		(pin "1"
 		)
@@
 			(at 304.8 44.45 90)
 			(effects
+				(font
+					(size 1.27 1.27)
+				)
+				(hide yes)
+			)
+		)
+		(property "FT Rotation Offset" "180"
+			(at 304.8 44.45 90)
+			(effects
