File: elec_2S_BMS_plus_charger/power.kicad_sch (KiCad schematic)
At the start: 45 parts, among them J1 JST -EH 2, J13 Dynamixel-3, J14 Dynamixel-3, J2 JST SH, J3 JST -EH 2, J4 JST -EH 2, J5 pico2, J6 pico2, J7 JST SH, Q1 BSZ034N04LS, Q2 BSZ034N04LS, U1 HY2120, U2 BQ25887RGE

Commit message: [update] Now running test on rasp zero 2W + HAT
Parts:
- L1: footprint Inductor_SMD:L_6.3x6.3_H3 -> LCSC_parts_lib:IND-SMD_L7.2-W6.6_GPSR0730
Changed lines of the file:
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@@
 			)
 		)
-		(property "Footprint" "Inductor_SMD:L_6.3x6.3_H3"
+		(property "Footprint" "LCSC_parts_lib:IND-SMD_L7.2-W6.6_GPSR0730"
 			(at 207.01 137.16 0)
 			(effects
